File: pcb/bb48-fdc.kicad_sch (KiCad schematic)
At the start: 10 parts, among them J1 FDD 34-pin host, J2 P2000T_EXPANSION_PORT, U1 74LS06, U2 74LS06, U3 74LVC14

Commit message: Revising design
Parts:
- added C5, C6, C7, C8: 0.1uF, Capacitor_SMD:C_0805_2012Metric, symbol Device:C
- added J4: Atmel-JTAG-10, Connector_IDC:IDC-Header_2x05_P2.54mm_Vertical, symbol atf1504_plcc44_breakout:Atmel-JTAG-10
- added R1, R2, R3, R4, R5: 1k, Resistor_SMD:R_0805_2012Metric, symbol Device:R_Small
- added U4: CY62128Exx-xxS, Package_SO:SOP-32_11.305x20.495mm_P1.27mm, symbol Memory_RAM:CY62128Exx-xxS
- added U5, U7: SN74LVC8T245, Package_SO:SOIC-24W_7.5x15.4mm_P1.27mm, symbol Logic_LevelTranslator:SN74LVC8T245
- added U6: ATF1502AS, Package_LCC:PLCC-44_THT-Socket, symbol atf1504as-plcc44:ATF1504AS-xJx44
- C1, C2, C3: value 100n -> 0.1uF
Connections:
- net +3V3: now also U5.23 (V_{CCB}), U5.24 (V_{CCB}), U7.23 (V_{CCB}), U7.24 (V_{CCB})
- net +5V: now also U4.30 (CS2/CE2), U4.32 (VCC), U5.1 (V_{CCA}), U7.1 (V_{CCA}), U7.2 (DIR)
- net GND: now also J2.1 (GND), C5.2, C6.2, C7.2, C8.2, J4.10 (GND), J4.2 (GND), U4.16 (GND), U5.11 (GND), U5.12 (GND), U5.13 (GND), U6.10 (GND), U6.22 (GND), U6.30 (GND), U6.42 (GND), U7.11 (GND), U7.12 (GND), U7.13 (GND), U7.22 (~{OE}); no longer U2.11, U2.13
- net ~{FDD_DSKCHG}: now also R4.1; no longer U3.9
- net ~{FDD_INDEX}: now also R1.1; no longer U3.1
- net ~{FDD_RDATA}: now also R3.1; no longer U3.5
- net ~{FDD_TRK0}: now also R2.1; no longer U3.3
- net ~{FDD_WPT}: now also R5.1; no longer U3.11
- net ~{INT}: now reaches U2.10
- net ~{INT}: now also J2.29 (~{INT})
- net ~{WAIT}: now reaches U2.12
- net ~{WAIT}: now also J2.32 (~{WAIT})
- net D7: now reaches J2.10 (D7)
- net D7: now also U4.21 (I/O7), U5.10 (A8), U6.14 (I/O)
- net A0: now reaches J2.11 (A0)
- net A0: now also U4.12 (A0), U6.16 (I/O), U7.3 (A1)
- net A1: now reaches J2.12 (A1)
- net A1: now also U4.11 (A1), U6.17 (I/O), U7.4 (A2)
- net A2: now reaches J2.13 (A2)
- net A2: now also U4.10 (A2), U6.18 (I/O)
- net A3: now reaches J2.14 (A3)
- net A3: now also U4.9 (A3), U6.19 (I/O)
- net A4: now reaches J2.15 (A4)
- net A4: now also U4.8 (A4), U6.20 (I/O)
- net A5: now reaches J2.16 (A5)
- net A5: now also U4.7 (A5), U6.21 (I/O)
- net A6: now reaches J2.17 (A6)
- net A6: now also U4.6 (A6), U6.24 (I/O)
- net A7: now reaches J2.18 (A7)
- net A7: now also U4.5 (A7), U6.25 (I/O/PD2)
- net A8: now reaches J2.19 (A8)
- net A8: now also U4.27 (A8)
- net A9: now reaches J2.20 (A9)
- net A9: now also U4.26 (A9)
- net A10: now reaches J2.21 (A10)
- net A10: now also U4.23 (A10)
- net A11: now reaches J2.22 (A11)
- net A11: now also U4.25 (A11)
- net A12: now reaches J2.23 (A12)
- net A12: now also U4.4 (A12)
- net A13: now reaches J2.24 (A13)
- net A13: now also U4.28 (A13)
- net A14: now reaches J2.25 (A14)
- net A14: now also U4.3 (A14)
- net RAMS2: now reaches J2.26 (RAMS2)
- net RAMS2: now also U6.26 (I/O)
- net ~{MRQ}: now reaches J2.27 (~{MRQ})
- net ~{MRQ}: now also U6.27 (I/O)
- net ~{RD}: now reaches J2.28 (~{RD})
- net ~{RD}: now also U4.24 (~{OE}), U5.2 (DIR), U6.28 (I/O), U7.5 (A3)
- net D0: now reaches J2.3 (D0)
- net D0: now also U4.13 (I/O0), U5.3 (A1), U6.4 (I/O)
- net ~{WR}: now reaches J2.30 (~{WR})
- net ~{WR}: now also U4.29 (~{WE}), U6.29 (I/O), U7.6 (A4)
- net ~{IORQ}: now reaches J2.31 (~{IORQ})
- net ~{IORQ}: now also U6.31 (I/O)
- net ~{M1}: now reaches J2.33 (~{M1})
- net ~{M1}: now also U6.33 (I/O)
- net ~{RES}: now reaches J2.34 (~{RES})
- net ~{RES}: now also U6.34 (I/O), U7.7 (A5)
- net ~{RFSH}: now reaches J2.36 (~{RFSH})
- net ~{RFSH}: now also U6.1 (I/GCLR)
- net ~{DEW}: now reaches J2.37 (~{DEW/R2425})
- net ~{DEW}: now also U7.10 (A8)
- net PHI: now reaches J2.38 (PHI)
- net PHI: now also U7.8 (A6)
- net PHI2: now reaches J2.39 (PHI2)
- net PHI2: now also U6.2 (I/OE2/GCLK2)
- net D1: now reaches J2.4 (D1)
- net D1: now also U4.14 (I/O1), U5.4 (A2), U6.5 (I/O)
- net T4M: now reaches J2.40 (T4M)
- net T4M: now also U6.43 (I/GCLK1)
- net D2: now reaches J2.5 (D2)
- net D2: now also U4.15 (I/O2), U5.5 (A3), U6.6 (I/O)
- net D3: now reaches J2.6 (D3)
- net D3: now also U4.17 (I/O3), U5.6 (A4), U6.8 (I/O)
- net D4: now reaches J2.7 (D4)
- net D4: now also U4.18 (I/O4), U5.7 (A5), U6.9 (I/O)
- net D5: now reaches J2.8 (D5)
- net D5: now also U4.19 (I/O5), U5.8 (A6), U6.11 (I/O/PD1)
- net D6: now reaches J2.9 (D6)
- net D6: now also U4.20 (I/O6), U5.9 (A7), U6.12 (I/O)
- net MCU_D1: now reaches A1.A10 (GPIO6/UEXT_SCK)
- net MCU_D1: now also U5.20 (B2)
- net MCU_D0: now reaches A1.A11 (GPIO7/UEXT_MOSI)
- net MCU_D0: now also U5.21 (B1)
- net ~{MCU_DEW}: now reaches A1.A16 (GPIO12)
- net ~{MCU_DEW}: now also U7.14 (B8)
- net ~{MCU_FDC_CS}: now reaches A1.A17 (GPIO13)
- net ~{MCU_FDC_CS}: now also U7.15 (B7)
- net MCU_PHI: now reaches A1.A18 (GPIO14)
- net MCU_PHI: now also U7.16 (B6)
- net ~{MCU_RES}: now reaches A1.A19 (GPIO15)
- net ~{MCU_RES}: now also U7.17 (B5)
- net ~{MCU_WR}: now reaches A1.A20 (GPIO16)
- net ~{MCU_WR}: now also U7.18 (B4)
- net ~{MCU_RD}: now reaches A1.A21 (GPIO17)
- net ~{MCU_RD}: now also U7.19 (B3)
- net MCU_A1: now reaches A1.A22 (GPIO18)
- net MCU_A1: now also U7.20 (B2)
- net MCU_A0: now reaches A1.A23 (GPIO19)
- net MCU_A0: now also U7.21 (B1)
- net MCU_READY: now reaches A1.A24 (GPIO20)
- net MCU_READY: now also U6.44 (I/OE1)
- net MCU_D7: now reaches A1.A4 (GPIO0/UEXT_TX)
- net MCU_D7: now also U5.14 (B8)
- net MCU_D6: now reaches A1.A5 (GPIO1/UEXT_RX)
- net MCU_D6: now also U5.15 (B7)
- net MCU_D5: now reaches A1.A6 (GPIO2/SDA(UEXT,QWIIC))
- net MCU_D5: now also U5.16 (B6)
- net MCU_D4: now reaches A1.A7 (GPIO3/SCL(UEXT,QWIIC))
- net MCU_D4: now also U5.17 (B5)
- net MCU_D3: now reaches A1.A8 (GPIO4/UEXT_MISO)
- net MCU_D3: now also U5.18 (B4)
- net MCU_D2: now reaches A1.A9 (GPIO5/UEXT_CS)
- net MCU_D2: now also U5.19 (B3)
- net INT_ASSERT: now reaches A1.B21 (GPIO41/ADC1)
- net INT_ASSERT: now also U2.11
- new net: R1.2, U3.1
- new net: R2.2, U3.3
- new net: R3.2, U3.5
- new net: R4.2, U3.9
- new net: R5.2, U3.11
- new net RAM_A15: U4.31 (A15), U6.39 (I/O)
- new net RAM_A16: U4.2 (A16), U6.40 (I/O)
- new net TCK: J4.1 (TCK), U6.32 (I/O/TCK)
- new net TDI: J4.9 (TDI), U6.7 (I/O/TDI)
- new net TDO: J4.3 (TDO), U6.38 (I/O/TDO)
- new net TMS: J4.5 (TMS), U6.13 (I/O/TMS)
- new net VCC: C5.1, C6.1, C7.1, C8.1, J4.4 (VccT), U6.15 (VCC), U6.23 (VCC), U6.3 (VCC), U6.35 (VCC)
- new net WAIT_ASSERT: U2.13, U6.41 (I/O/GCLK3)
- new net ~{FDC_CS}: U5.22 (~{OE}), U6.37 (I/O), U7.9 (A7)
- new net ~{RAM_CS}: U4.22 (~{CS1}/~{CE1}), U6.36 (I/O)
- no-connect marks 41 -> 23
Other:
- moved on the sheet: C1, C2, C3, C4, U2E, U2F

Commit message: Cleaning up schematic
Parts:
- removed C1, C2, C3: 0.1uF, Capacitor_SMD:C_0603_1608Metric, symbol FDC_Interface:C
- removed C4: 4.7u, Capacitor_SMD:C_0805_2012Metric, symbol FDC_Interface:C
- removed C5, C6, C7, C8: 0.1uF, Capacitor_SMD:C_0805_2012Metric, symbol Device:C
- removed J2: P2000T_EXPANSION_PORT, Connector_PinHeader_2.54mm:PinHeader_2x20_P2.54mm_Vertical, symbol P2000T:P2000T_EXPANSION_PORT
- removed J4: Atmel-JTAG-10, Connector_IDC:IDC-Header_2x05_P2.54mm_Vertical, symbol atf1504_plcc44_breakout:Atmel-JTAG-10
- removed U4: CY62128Exx-xxS, Package_SO:SOP-32_11.305x20.495mm_P1.27mm, symbol Memory_RAM:CY62128Exx-xxS
- removed U5, U7: SN74LVC8T245, Package_SO:SOIC-24W_7.5x15.4mm_P1.27mm, symbol Logic_LevelTranslator:SN74LVC8T245
- removed U6: ATF1502AS, Package_LCC:PLCC-44_THT-Socket, symbol atf1504as-plcc44:ATF1504AS-xJx44
Connections:
- net WAIT_ASSERT is gone; now on net FDC_SIDE1: U2.13
- net ~{INT} is gone; now on net ~{FDD_WGATE}: U2.10
- net ~{WAIT} is gone; now on net ~{FDD_SIDE1}: U2.12
- net FDC_DIR: now also U1.13; no longer U1.9
- net FDC_DRVSA: now also U2.1; no longer U1.11
- net FDC_DRVSB: now also U1.9; no longer U1.3
- net FDC_MOTEA: now also U2.3; no longer U1.13
- net FDC_MOTEB: now also U1.11; no longer U1.5
- net FDC_SIDE1: no longer U2.9
- net FDC_STEP: now also U2.5; no longer U2.1
- net FDC_WDATA: now also U2.9; no longer U2.3
- net FDC_WGATE: now also U2.11; no longer U2.5
- net GND: now also J1.3
- net ~{FDD_DIR}: now also U1.12; no longer U1.8
- net ~{FDD_DRVSA}: now also U2.2; no longer U1.10
- net ~{FDD_DRVSB}: now also U1.8; no longer U1.4
- net ~{FDD_MOTEA}: now also U2.4; no longer U1.12
- net ~{FDD_MOTEB}: now also U1.10; no longer U1.6
- net ~{FDD_SIDE1}: no longer U2.8
- net ~{FDD_STEP}: now also U2.6; no longer U2.2
- net ~{FDD_WDATA}: now also U2.8; no longer U2.4
- net ~{FDD_WGATE}: no longer U2.6
- net INT_ASSERT: no longer names the net of A1.B21 (GPIO41/ADC1)
- net INT_ASSERT: no longer U2.11
- net MCU_A0: no longer names the net of A1.A23 (GPIO19)
- net MCU_A1: no longer names the net of A1.A22 (GPIO18)
- net MCU_D0: no longer names the net of A1.A11 (GPIO7/UEXT_MOSI)
- net MCU_D1: no longer names the net of A1.A10 (GPIO6/UEXT_SCK)
- net MCU_D2: no longer names the net of A1.A9 (GPIO5/UEXT_CS)
- net MCU_D3: no longer names the net of A1.A8 (GPIO4/UEXT_MISO)
- net MCU_D4: no longer names the net of A1.A7 (GPIO3/SCL(UEXT,QWIIC))
- net MCU_D5: no longer names the net of A1.A6 (GPIO2/SDA(UEXT,QWIIC))
- net MCU_D6: no longer names the net of A1.A5 (GPIO1/UEXT_RX)
- net MCU_D7: no longer names the net of A1.A4 (GPIO0/UEXT_TX)
- net MCU_PHI: no longer names the net of A1.A18 (GPIO14)
- net MCU_READY: no longer names the net of A1.A24 (GPIO20)
- net ~{MCU_DEW}: no longer names the net of A1.A16 (GPIO12)
- net ~{MCU_FDC_CS}: no longer names the net of A1.A17 (GPIO13)
- net ~{MCU_RD}: no longer names the net of A1.A21 (GPIO17)
- net ~{MCU_RES}: no longer names the net of A1.A19 (GPIO15)
- net ~{MCU_WR}: no longer names the net of A1.A20 (GPIO16)
- no-connect marks 23 -> 36
Other:
- moved on the sheet: R1, R2, R3, R4, R5, U1A, U1B, U1C, U1D, U1E, U1F, U1G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

Commit message: Initial design PCB
Parts:
- removed R1, R2, R3, R4, R5: 1k, Resistor_SMD:R_0805_2012Metric, symbol Device:R_Small
- added C1, C2, C3: 0.1uF, Capacitor_SMD:C_0805_2012Metric_Pad1.18x1.45mm_HandSolder, symbol Device:C_Small
- added H1, H2, H3, H4: MountingHole, symbol Mechanical:MountingHole
- added RN1, RN2, RN3: 1k, Resistor_THT:R_Array_SIP7, symbol Device:R_Network06_Split
- U3: value 74LVC14 -> 74LVC14A
- renumbered U2 to U1, U1 to U2
Connections:
- net ~{FDD_RDATA} is gone; now on net ~{FDD_READ_DATA}: J1.30 (~{READ_DATA})
- net +3V3: now also C1.1
- net +5V: now also C2.1, C3.1, RN1.1 (R1), RN1.1 (R1), RN1.1 (R1), RN1.1 (R1), RN1.1 (R1), RN1.1 (R1)
- net FDC_INDEX: now also U3.8; no longer U3.2
- net FDC_STEP: now also U2.1, RN2.4 (R3.2); no longer U2.5
- net GND: now also U1.1, U3.3, C1.2, C2.2, C3.2, RN2.1 (R1), RN2.1 (R1), RN2.1 (R1), RN2.1 (R1), RN2.1 (R1), RN2.1 (R1), RN3.1 (R1), RN3.1 (R1), RN3.1 (R1), RN3.1 (R1), RN3.1 (R1), RN3.1 (R1); no longer U3.13
- net ~{FDD_INDEX}: now also U3.9, RN1.2 (R1.2)
- net ~{FDD_STEP}: now also U2.2; no longer U2.6
- net ~{FDD_DS3} / NC: now reaches J1.6 (~{DS3}_/_NC)
- net ~{FDD_DS3} / NC: now also U1.6
- net FDC_DS3: now reaches U1.5
- net FDC_DS3: now also A1.B20 (GPIO40/ADC0), RN3.4 (R3.2)
- net ~{FDD_READ_DATA}: now reaches U3.5
- net ~{FDD_READ_DATA}: now also RN1.6 (R5.2)
- net FDC_DENSITY_SELECT: now reaches A1.B21 (GPIO41/ADC1)
- net FDC_DENSITY_SELECT: now also U1.3, RN3.3 (R2.2)
- removed net FDC_DENSEL: A1.B20 (GPIO40/ADC0), U1.1
- net FDC_DIR renamed FDC_DIRECTION
- net FDC_DIRECTION: now also U2.3, RN2.3 (R2.2); no longer U2.13
- net FDC_DRVSA renamed FDC_DRIVE_A_DS2
- net FDC_DRIVE_A_DS2: now also U1.11, RN3.7 (R6.2); no longer U1.1
- net FDC_DRVSB renamed FDC_DRIVE_B_DS1
- net FDC_DRIVE_B_DS1: now also U1.13, RN3.6 (R5.2); no longer U1.9
- net FDC_DSKCHG renamed FDC_DISK_CHANGE_READY
- net FDC_DISK_CHANGE_READY: now also U3.2; no longer U3.8
- net FDC_MOTEA renamed FDC_MOTOR_A_DS0
- net FDC_MOTOR_A_DS0: now also U1.9, RN3.5 (R4.2); no longer U1.3
- net FDC_MOTEB renamed FDC_MOTOR_B_MOTOR_ON
- net FDC_MOTOR_B_MOTOR_ON: now also U2.5, RN2.2 (R1.2); no longer U2.11
- net FDC_RDATA renamed FDC_READ_DATA
- net FDC_SIDE1 renamed FDC_SIDE_1
- net FDC_SIDE_1: now also RN2.7 (R6.2)
- net FDC_TRK0 renamed FDC_TRACK_0
- net FDC_TRACK_0: now also U3.10; no longer U3.4
- net FDC_WDATA renamed FDC_WRITE_DATA
- net FDC_WRITE_DATA: now also RN2.5 (R4.2)
- net FDC_WGATE renamed FDC_WRITE_GATE
- net FDC_WRITE_GATE: now also RN2.6 (R5.2)
- net FDC_WPT renamed FDC_WRITE_PROTECT
- net FDC_WRITE_PROTECT: now also U3.12; no longer U3.10
- net ~{FDD_DENSEL} renamed ~{FDD_DENSITY_SELECT} / ~{FDD_DISK_CHANGE} / NC
- net ~{FDD_DENSITY_SELECT} / ~{FDD_DISK_CHANGE} / NC: now also U1.4; no longer U1.2
- net ~{FDD_DIR} renamed ~{FDD_DIRECTION}
- net ~{FDD_DIRECTION}: now also U2.4; no longer U2.12
- net ~{FDD_DRVSA} renamed ~{FDD_DRIVE_A} / ~{FDD_DS2}
- net ~{FDD_DRIVE_A} / ~{FDD_DS2}: now also U1.10; no longer U1.2
- net ~{FDD_DRVSB} renamed ~{FDD_DRIVE_B} / ~{FDD_DS1}
- net ~{FDD_DRIVE_B} / ~{FDD_DS1}: now also U1.12; no longer U1.8
- net ~{FDD_DSKCHG} renamed ~{FDD_DISK_CHANGE} / ~{FDD_READY}
- net ~{FDD_DISK_CHANGE} / ~{FDD_READY}: now also U3.1, RN1.7 (R6.2)
- net ~{FDD_MOTEA} renamed ~{FDD_MOTOR_A} / ~{FDD_DS0}
- net ~{FDD_MOTOR_A} / ~{FDD_DS0}: now also U1.8; no longer U1.4
- net ~{FDD_MOTEB} renamed ~{FDD_MOTOR_B} / ~{FDD_MOTOR_ON}
- net ~{FDD_MOTOR_B} / ~{FDD_MOTOR_ON}: now also U2.6; no longer U2.10
- net ~{FDD_SIDE1} renamed ~{FDD_SIDE_1}
- net ~{FDD_TRK0} renamed ~{FDD_TRACK_0}
- net ~{FDD_TRACK_0}: now also U3.11, RN1.4 (R3.2)
- net ~{FDD_WDATA} renamed ~{FDD_WRITE_DATA}
- net ~{FDD_WGATE} renamed ~{FDD_WRITE_GATE}
- net ~{FDD_WPT} renamed ~{FDD_WRITE_PROTECT}
- net ~{FDD_WRITE_PROTECT}: now also U3.13, RN1.5 (R4.2)
- no-connect marks 36 -> 38
Other:
- moved on the sheet: A1, J1, U1A, U1B, U1C, U1D, U1E, U1F, U1G, U2A, U2B, U2C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
